File: PoE-IP-Camera/Power and PoE.kicad_sch (KiCad schematic)
At the start: 92 parts, among them J1 RJ45, J2 Barrel_Jack_MountingPin, P1 USB_C_Plug_USB2.0, SW1 SW_DIP_x03, T1 SM51625EL, U1 TPS54260DGQ, U2 TLP293, U3 CJ431

Commit message: частичная трассировка
Connections:
- net IN1+: now reaches J1.1, T1.23 (MX1+)
- net IN1-: now reaches J1.2, T1.22 (MX1-)
- net IN2+: now reaches J1.3, T1.20 (MX2+)
- net IN2-: now reaches J1.4, T1.19 (MX2-)
- net IN3+: now reaches J1.5, T1.17 (MX3+)
- net IN3-: now reaches J1.6, T1.16 (MX3-)
- net IN4+: now reaches J1.7, T1.14 (MX4+)
- net IN4-: now reaches J1.8, T1.13 (MX4-)
Other:
- moved on the sheet: D1, D2

Commit message: чут чут трассировки
Parts:
- added R21: 1k, Resistor_SMD:R_0402_1005Metric, symbol Device:R
- renumbered R21 to R22, R22 to R23, R23 to R24, R24 to R25, R25 to R26, R26 to R27, R27 to R28, R28 to R29, R29 to R30, R30 to R31, R31 to R32, R32 to R33, R33 to R34, R34 to R35
Connections:
- net GND1: now also PS1.1 (RSNS), R21.1
- net at PS1.8 (CS): now also R21.2
