File: PoE-IP-Camera/PoE-IP-Camera.kicad_pcb (KiCad board)
At the start: 2 copper layers, 72.9 x 77.5 mm, 139 parts, among them J1 RJ45, J2 Barrel_Jack_MountingPin, J3 Conn_01x0, J4 Conn_01x04_Socket, J5 Conn_01x04_Socket, P1 USB_C_Plug_USB2.0, SW1 SW_DIP_x03, SW2 434133025816, T1 SM51625EL, U1 TPS54260DGQ, U2 TLP293, U3 CJ431, U5 STM32F030F4Px, Y1 X322525MOB4SI, Y2 X322525MOB4SI

Commit message: частичная трассировка
Parts:
- moved R18 0.21 mm to (78.0, 76.2)
- moved C18 0.20 mm to (80.0, 75.2)
- turned C4 to -90 degrees
Connections:
- net Net-(T1-MX1+) renamed IN1+
- net Net-(T1-MX1-) renamed IN1-
- net Net-(T1-MX2+) renamed IN2+
- net Net-(T1-MX2-) renamed IN2-
- net Net-(T1-MX3+) renamed IN3+
- net Net-(T1-MX3-) renamed IN3-
- net Net-(T1-MX4+) renamed IN4+
- net Net-(T1-MX4-) renamed IN4-
- net Net-(T1-TCT4) renamed hehe
- U5 pad 18: unconnected-(U5-PA10-Pad18) -> EMAC_CRS_DV
Routing:
- net UART_STM_RX: track 0.00 -> 73.6 mm
- net UART_STM_TX: track 0.00 -> 71.3 mm
- net Net-(J3-Pin_1): track 0.00 -> 57.9 mm, vias 0 -> 1
- net EMAC_RXD0: track 0.00 -> 44.0 mm
- net RST: track 0.00 -> 44.0 mm, vias 0 -> 2
- net EMAC_CRS_DV: track 0.00 -> 43.8 mm
- net MDI_0: track 0.00 -> 42.5 mm
- net EMAC_MDC: track 0.00 -> 42.2 mm
- net EMAC_RXD1: track 0.00 -> 40.2 mm
- net EMAC_TX_EN: track 0.00 -> 39.8 mm
- net EMAC_TXD1: track 0.00 -> 36.9 mm
- net EMAC_TXD0: track 0.00 -> 36.3 mm
- net SW_CLK: track 0.00 -> 28.2 mm
- net SW_DIO: track 0.00 -> 27.4 mm
- net IN4+: track 0.00 -> 26.5 mm
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- added copper zone on F.Cu, net /Power and PoE/POE_IN_+
- added copper zone on F.Cu, net /Power and PoE/POE_VAC1
- added copper zone on F.Cu, net /Power and PoE/POE_VAC2
- added copper zone on F.Cu, net /Power and PoE/POE_VAC3
- added copper zone on F.Cu, net /Power and PoE/POE_VAC4
- added copper zone on F.Cu, net Net-(D10-A)
- added copper zone on F.Cu, net Net-(D10-K)
- added copper zone on B.Cu, net Net-(D12-K)
- added copper zone on F.Cu, net Net-(D12-K)
- added copper zone on B.Cu, net Net-(D9-A)
- added copper zone on F.Cu, net Net-(D9-A)
- added copper zone on F.Cu, net Net-(PS1-AUX_V)
- added copper zone on F.Cu, net Net-(U1-VIN)
Other:
- copper layers 2 -> 4

Commit message: чут чут трассировки
Parts:
- added R21: 1k, Resistor_SMD:R_0402_1005Metric, F.Cu at (51.7, 48.5)
- renumbered R21 to R22, R22 to R23, R23 to R24, R24 to R25, R25 to R26, R26 to R27, R27 to R28, R28 to R29, R29 to R30, R30 to R31, R31 to R32, R32 to R33, R33 to R34, R34 to R35, R35 to R36, R36 to R37, R37 to R38, R38 to R39, R39 to R40, R40 to R41, R41 to R42, R42 to R43, R43 to R44, R44 to R45, R45 to R46, R46 to R47, R47 to R48, R48 to R49, R49 to R50
Connections:
- net hehe renamed Net-(T1-TCT4)
- PS1 pad 1: unconnected-(PS1-RSNS-Pad1) -> GND1
- PS1 pad 8: unconnected-(PS1-CS-Pad8) -> Net-(PS1-CS)
- U1 pad 11: Earth -> (no net)
Routing:
- net Net-(DD1-LED0/_PHYAD[0]/PMEB): track 15.7 -> 75.2 mm, vias 0 -> 2
- net Net-(DD1-LED1/PHYAD[1]): track 20.1 -> 76.8 mm, vias 0 -> 2
- net RST: track 44.0 -> 72.2 mm, vias 2 -> 3
- net /Power and PoE/POE_IN_-: track 0.00 -> 14.8 mm, vias 0 -> 16
- net Net-(PS1-CS): track 0.00 -> 9.79 mm, vias 0 -> 2
- net Net-(U1-VIN): track 0.00 -> 6.22 mm
- net Net-(PS1-FB): track 4.66 -> 9.50 mm
- net Net-(P1-VCONN): track 0.00 -> 3.28 mm
- net /Power and PoE/POE_IN_+: track 0.00 -> 3.21 mm, vias 10 -> 29
- net Net-(P1-CC): track 0.00 -> 1.99 mm
- net Net-(R31-Pad2): track 0.00 -> 1.81 mm
- net Net-(JP1-A): track 19.5 -> 21.2 mm
- net +3.3V: track 24.0 -> 25.4 mm, vias 4 -> 5
- net +12V_POE: track 0.00 -> 0.55 mm, vias 0 -> 1
- net Net-(DD1-AVDD33_1): vias 0 -> 5
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- added copper zone on F.Cu, net +12V_POE
- added copper zone on B.Cu, net /Power and PoE/POE_IN_+
- added copper zone on B.Cu, net /Power and PoE/POE_IN_-
- added copper zone on F.Cu, net /Power and PoE/POE_IN_-
- added copper zone on In2.Cu, net /Power and PoE/POE_IN_-
- added copper zone on F.Cu, net GND1
- added copper zone on In1.Cu, net GND1
- added copper zone on F.Cu, net Net-(D14-A)
- added copper zone on F.Cu, net Net-(D9-K)
- added copper zone on In2.Cu, net Net-(DD1-AVDD33_1)
- added copper zone on F.Cu, net Net-(PS1-CP)
- added copper zone on In2.Cu, net Net-(PS1-CP)

Commit message: Завершение трассировки
Parts:
- added G***: LOGO, LOGO, F.Cu at (43.9, 104.7)
- added G***: LOGO, LOGO, B.Cu at (74.5, 58.9)
- added G***: LOGO, LOGO, B.Cu at (59.2, 49.0)
- added G***: LOGO, LOGO, B.Cu at (62.0, 96.4)
- added G***: LOGO, LOGO, B.Cu at (47.4, 53.8)
- added G***: LOGO, LOGO, F.Cu at (23.9, 102.0)
- added G***: LOGO, LOGO, F.Cu at (80.7, 102.5)
- added G***: LOGO, LOGO, F.Cu at (25.8, 85.3)
- added G***: LOGO, LOGO, B.Cu at (26.6, 111.3)
- added G***: LOGO, LOGO, B.Cu at (27.1, 101.3)
- added G***: LOGO, LOGO, B.Cu at (57.4, 70.9)
- added G***: LOGO, LOGO, B.Cu at (68.0, 51.4)
- added G***: LOGO, LOGO, B.Cu at (38.6, 51.3)
- added kibuzzard-67A498E6: G***, kibuzzard-67A498E6, F.Cu at (73.5, 95.0)
- added kibuzzard-67A49B3B: G***, kibuzzard-67A49B3B, F.Cu at (78.0, 97.6)
- added kibuzzard-67A49B47: G***, kibuzzard-67A49B47, F.Cu at (64.0, 97.6)
Connections:
- REF** pad 1: (no net) -> Earth
- U1 pad 11: (no net) -> Earth
Routing:
- net +12V_POE: track 0.55 -> 87.2 mm, vias 1 -> 17
- net +3.3V: track 25.4 -> 68.9 mm, vias 5 -> 26
- net Earth: track 10.4 -> 31.3 mm, vias 0 -> 78
- net Net-(D10-A): track 0.91 -> 5.63 mm
- net Net-(D10-K): track 0.00 -> 4.67 mm
- net GND1: track 0.00 -> 2.72 mm, vias 0 -> 59
- net +5V USB: track 14.4 -> 15.2 mm, vias 0 -> 6
- net Net-(PS1-CP): track 0.00 -> 0.70 mm
- net Net-(U1-VIN): track 6.22 -> 6.39 mm, vias 4 -> 5
- added copper zone on In2.Cu, net +12V_POE
- added copper zone on F.Cu, net +3.3V
- added copper zone on In2.Cu, net +3.3V
- added copper zone on In2.Cu, net +5V USB
- added copper zone on B.Cu, net Earth
- added copper zone on F.Cu, net Earth
- added copper zone on In1.Cu, net Earth
- added copper zone on B.Cu, net Net-(U1-VIN)
- added copper zone on In2.Cu, net VIN
Other:
- board size 72.9 x 77.5 mm -> 73 x 77.5 mm
- board text added: "+3.3"
- board text added: "CLK"
- board text added: "DC in 4.2-13V"
- board text added: "DIO"
- board text added: "ESP32 Cam"
- board text added: "GND"
- board text added: "PoE"
- board text added: "PoE 13W Type 1 PD"
- board text added: "RX"
- board text added: "TX"
- board text added: "USB"
- board text added: "USB-C PWR in"
- board text added: "VIN"
